File: PCB/Kicad_project/OPA_Alice_ECM_Microphone.kicad_pcb (KiCad board)
At the start: 2 copper layers, 38.8 x 75 mm, 46 parts, among them J1 XLR, J6 Conn_01x01_Pin, J7 Conn_01x01_Pin, J8 Conn_01x01_Pin, J9 Conn_01x01_Pin, U1 OPA1642AIDR, U2 TL431DBZ

Commit message: 新增BOM
Parts:
- removed ? (x16): , 
- removed J6, J7, J8, J9: Conn_01x01_Pin, custom_connector:F5-9-0.4直筒内绕平行针_触摸弹簧
- removed U2: TL431DBZ, Package_TO_SOT_SMD:SOT-23
- added J2: Conn_01x01_Pin, custom_connector:F5-9-0.4直筒内绕平行针_触摸弹簧, F.Cu at (148.6, 122.2)
- added J3: Conn_01x01_Pin, custom_connector:F5-9-0.4直筒内绕平行针_触摸弹簧, F.Cu at (148.6, 54.2)
- added J4: Conn_01x01_Pin, custom_connector:F5-9-0.4直筒内绕平行针_触摸弹簧, F.Cu at (120.6, 122.2)
- added J5: XLR, Connector_Molex:Molex_PicoBlade_53398-0371_1x03-1MP_P1.25mm_Vertical, F.Cu at (122.3, 105.1)
- added TL431: TL431DBZ, Package_TO_SOT_SMD:SOT-23, F.Cu at (147.3, 85.5)
- J1: value XLR -> Conn_01x01_Pin; footprint Connector_JST:JST_XH_B3B-XH-A_1x03_P2.50mm_Vertical -> custom_connector:F5-9-0.4直筒内绕平行针_触摸弹簧
- MK1: footprint Connector_JST:JST_XH_B2B-XH-A_1x02_P2.50mm_Vertical -> Connector_Molex:Molex_PicoBlade_53398-0271_1x02-1MP_P1.25mm_Vertical
- moved J1 48.7 mm to (120.6, 54.2), turned to 90 degrees
- moved R7 10.6 mm to (147.2, 82.4), turned to 180 degrees
- moved D1 5.89 mm to (146.2, 89.6), turned to 180 degrees
- moved R8 5.71 mm to (143.8, 85.6)
- moved MK1 1.32 mm to (134.6, 63.1)
- moved R5 1.22 mm to (147.2, 80.4), turned to 180 degrees
- moved C8 1.04 mm to (130.8, 107.2)
- moved C9 1.04 mm to (128.1, 107.2)
- moved C6 0.30 mm to (145.3, 98.6)
Connections:
- J1 pad 1: /XLR_3 -> GND
Routing:
- net VCC: track 46.9 -> 33.2 mm
- net GND: track 17.1 -> 24.9 mm
- net +12V: track 28.5 -> 26.1 mm
- net Net-(C4-Pad1): track 11.7 -> 10.5 mm
- net Net-(C5-Pad1): track 15.1 -> 14.1 mm
- net /Signal_Output_-: track 26.5 -> 27.4 mm
- net /XLR_3: track 11.5 -> 10.8 mm
Other:
- board text added: "Option"
- board text added: "Sig- Sig+ GND"
- board text removed: "Alice OPA ECM Mic Board"
- board text removed: "Sig+ Sig- GND"
