File: PCB/Kicad_project/OPA_Alice_ECM_Microphone.kicad_sch (KiCad schematic)
At the start: 30 parts, among them J1 XLR, J6 Conn_01x01_Pin, J7 Conn_01x01_Pin, J8 Conn_01x01_Pin, J9 Conn_01x01_Pin, U1 OPA1642AIDR, U2 TL431DBZ

Commit message: 新增BOM
Parts:
- removed J1: XLR, Connector_JST:JST_XH_B3B-XH-A_1x03_P2.50mm_Vertical, symbol Connector:Conn_01x03_Pin
- added J5: XLR, Connector_Molex:Molex_PicoBlade_53398-0371_1x03-1MP_P1.25mm_Vertical, symbol Connector:Conn_01x04_Pin
- MK1: footprint Connector_JST:JST_XH_B2B-XH-A_1x02_P2.50mm_Vertical -> Connector_Molex:Molex_PicoBlade_53398-0271_1x02-1MP_P1.25mm_Vertical
- R7: value 38k -> 39k
- renumbered J9 to J1, J8 to J2, J7 to J3, J6 to J4
Connections:
- net GND: now also MK1.MP, J5.1 (Pin_1), J5.MP (Pin_4)
- net XLR_2: now also J5.2 (Pin_2)
- net XLR_3: now also J5.3 (Pin_3)
Other:
- note added: "Vout = (1+R7/R8) x Vref"
- note added: "≈ 12.25V"
- note added: "实测 ≈ 11.5V"
- note removed: "Vout = (1+R1/R2) x Vref"
- moved on the sheet: J1, J2, J3, J4, R1, R10, R9
